File: hardware/mainboard/mainboard.kicad_pcb (KiCad board)
At the start: 2 copper layers, 48 x 34 mm, 40 parts, among them IC1 MP2338GTL-Z, J1 USB_C_Receptacle_USB2.0_16P, Q1 Q_PMOS_DGS, U1 ESP32-C6-MINI-1, U2 BMI323, U3 LSM6DS3

Commit message: rev1
Parts:
- removed R_I2C1, R_I2C2, R_SPI1: 0, Resistor_SMD:R_0603_1608Metric_Pad0.98x0.95mm_HandSolder
- removed R_SPI2: 47k, Resistor_SMD:R_0603_1608Metric_Pad0.98x0.95mm_HandSolder
- moved FID1 23.8 mm to (136.8, 68.5)
- moved C2 11.7 mm to (138.8, 63.6)
- moved C1 11.6 mm to (138.8, 61.1)
- moved C4 11.2 mm to (138.8, 58.5)
- moved C3 11.2 mm to (138.8, 55.9)
- moved U2 11.1 mm to (136.3, 62.6)
- moved U3 10.7 mm to (136.4, 57.1)
- moved R_SCL1 7.39 mm to (133.8, 61.4)
- moved R_SDA1 5.95 mm to (132.3, 61.4)
- moved Q1 4.83 mm to (134.3, 54.1)
- moved C7 3.59 mm to (119.6, 66.6)
- moved IC1 3.59 mm to (116.5, 66.8)
- moved C10 3.59 mm to (117.7, 59.4)
- moved C8 3.59 mm to (117.4, 63.0)
- moved C9 3.59 mm to (122.2, 62.4)
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- renumbered FID2 to FID1
Connections:
- U1 pad 20: BMI323_INT2 -> CHIPSEL
- U1 pad 22: LSM_INT2 -> BMI323_INT2
- U1 pad 27: CHIPSEL -> CHIPSEL_LSM
- U1 pad 28: CHIPSEL_LSM -> LSM_INT2
- U2 pad 12: Net-(U2-CSB) -> CHIPSEL
Routing:
- net GND: track 99.4 -> 61.8 mm, vias 11 -> 12
- net VDD: track 56.7 -> 32.5 mm, vias 0 -> 2
- net BMI323_INT2: track 30.6 -> 11.3 mm, vias 2 -> 0
- net SCL/SCK: track 31.4 -> 13.3 mm, vias 0 -> 2
- net SDI/SDA: track 31.6 -> 14.1 mm
- net CHIPSEL_LSM: track 21.9 -> 5.55 mm
- net SDO/SA0: track 29.6 -> 13.4 mm
- net LSM_INT2: track 22.0 -> 6.98 mm, vias 2 -> 0
- net BMI323_INT1: track 28.6 -> 15.4 mm
- net LSM_INT1: track 21.8 -> 9.98 mm, vias 2 -> 0
- net Net-(U2-CSB): track 10.3 -> 0.00 mm, vias 2 -> 0
- net VAA: track 10.0 -> 18.0 mm
- net +3V3: track 29.5 -> 25.0 mm, vias 2 -> 3
- net CHIPSEL: track 9.90 -> 11.1 mm
- net IMU_EN: track 3.25 -> 2.73 mm
Other:
- board size 48 x 34 mm -> 32 x 34 mm

Commit message: mainboard edits
Parts:
- C1, C10, C11, C12, C2, C3, C4, C5, C6, C7, C8, C9: footprint Capacitor_SMD:C_0504_1310Metric_Pad0.83x1.28mm_HandSolder -> Capacitor_SMD:C_0504_1310Metric
- D2: footprint Diode_SMD:D_0805_2012Metric_Pad1.15x1.40mm_HandSolder -> Diode_SMD:D_0805_2012Metric
- R1, R10, R2, R3, R4, R5, R6, R7, R8, R9, R_SCL1, R_SDA1: footprint Resistor_SMD:R_0603_1608Metric_Pad0.98x0.95mm_HandSolder -> Resistor_SMD:R_0603_1608Metric

Commit message: mainboard edits
Parts:
- removed the FID1 at (136.8, 68.5)
- removed the FID1 at (132.0, 69.0)
- added FID1: Fiducial, Fiducial:Fiducial_0.5mm_Mask1.5mm, F.Cu at (1.02, 1.02)
- C1, C10, C11, C12, C2, C3, C4, C5, C6, C7, C8, C9: footprint Capacitor_SMD:C_0504_1310Metric -> Capacitor_SMD:C_0402_1005Metric
