File: mainboard/mainboard_mk1.kicad_sch (KiCad schematic)
At the start: 13 parts, among them J1 Conn_01x03_Pin, J2 Conn_01x03_Pin, J3 Conn_01x03_Pin, J4 Conn_01x03_Pin, J5 align2, J6 Conn_01x05_Pin, J7 Conn_01x02_Pin, J8 IMU, J9 align1, U1 74LS04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

Commit message: mk1 3d view done
Parts:
- J6: footprint Connector_PinHeader_2.54mm:PinHeader_1x05_P2.54mm_Vertical -> Connector_PinHeader_2.54mm:PinHeader_1x06_P2.54mm_Horizontal
Changed lines of the file:
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@@
 			)
 		)
-		(property "Footprint" "Connector_PinHeader_2.54mm:PinHeader_1x05_P2.54mm_Vertical"
+		(property "Footprint" "Connector_PinHeader_2.54mm:PinHeader_1x06_P2.54mm_Horizontal"
 			(at 161.29 91.44 0)
 			(effects
